Commit message: first

File: urdf/ASK-4.urdf (robot description, URDF)
Before this commit: robot ASK-4, 13 links, 11 joints
Links:
- added link FL_foot_link, mass 0.0332506166455944; collision mesh filename=package://ASK-4-2/meshes/FL_foot_link.STL; visual mesh filename=package://ASK-4-2/meshes/FL_foot_link.STL
- added link FR_foot_link, mass 0.0332506166455944; collision mesh filename=package://ASK-4-2/meshes/FR_foot_link.STL; visual mesh filename=package://ASK-4-2/meshes/FR_foot_link.STL
- added link RL_foot_link, mass 0.0332506166455944; collision mesh filename=package://ASK-4-2/meshes/RL_foot_link.STL; visual mesh filename=package://ASK-4-2/meshes/RL_foot_link.STL
- added link RR_foot_link, mass 0.0332506166455944; collision mesh filename=package://ASK-4-2/meshes/RR_foot_link.STL; visual mesh filename=package://ASK-4-2/meshes/RR_foot_link.STL
- link FL_calf_link: mass 0.2303901 -> 0.196508884495562; geometry collision mesh filename=package://ASK-4-2/meshes/FL_calf_link.STL; visual mesh filename=package://ASK-4-2/meshes/FL_calf_link.STL
- link FL_hip_link: mass 0.3376556  -> 0.337654873921649; geometry collision mesh filename=package://ASK-4-2/meshes/FL_hip_link.STL; visual mesh filename=package://ASK-4-2/meshes/FL_hip_link.STL
- link FL_thigh_link: mass  0.9885170 -> 0.98851736736006; geometry collision mesh filename=package://ASK-4-2/meshes/FL_thigh_link.STL; visual mesh filename=package://ASK-4-2/meshes/FL_thigh_link.STL
- link FR_calf_link: mass 0.2303901 -> 0.196508884495563; geometry collision mesh filename=package://ASK-4-2/meshes/FR_calf_link.STL; visual mesh filename=package://ASK-4-2/meshes/FR_calf_link.STL
- link FR_hip_link: mass  0.3376577  -> 0.337657104489193; geometry collision mesh filename=package://ASK-4-2/meshes/FR_hip_link.STL; visual mesh filename=package://ASK-4-2/meshes/FR_hip_link.STL
- link FR_thigh_link: mass 0.9817966 -> 0.981796539065317; geometry collision mesh filename=package://ASK-4-2/meshes/FR_thigh_link.STL; visual mesh filename=package://ASK-4-2/meshes/FR_thigh_link.STL
- link RL_calf_link: mass 0.2303901 -> 0.196508884495564; geometry collision mesh filename=package://ASK-4-2/meshes/RL_calf_link.STL; visual mesh filename=package://ASK-4-2/meshes/RL_calf_link.STL
- link RL_hip_link: mass  0.3376556 -> 0.33765486830875; geometry collision mesh filename=package://ASK-4-2/meshes/RL_hip_link.STL; visual mesh filename=package://ASK-4-2/meshes/RL_hip_link.STL
- link RL_thigh_link: mass 0.9885474  -> 0.988547565628563; geometry collision mesh filename=package://ASK-4-2/meshes/RL_thigh_link.STL; visual mesh filename=package://ASK-4-2/meshes/RL_thigh_link.STL
- link RR_calf_link: mass  0.2303901 -> 0.196508883743766; geometry collision mesh filename=package://ASK-4-2/meshes/RR_calf_link.STL; visual mesh filename=package://ASK-4-2/meshes/RR_calf_link.STL
- link RR_hip_link: mass  0.3376577  -> 0.337657104489195; geometry collision mesh filename=package://ASK-4-2/meshes/RR_hip_link.STL; visual mesh filename=package://ASK-4-2/meshes/RR_hip_link.STL
- link RR_thigh_link: mass  0.9817966  -> 0.981796539186015; geometry collision mesh filename=package://ASK-4-2/meshes/RR_thigh_link.STL; visual mesh filename=package://ASK-4-2/meshes/RR_thigh_link.STL
- link base_link: mass 5.1396761  -> 5.13967166144139; geometry collision mesh filename=package://ASK-4-2/meshes/base_link.STL; visual mesh filename=package://ASK-4-2/meshes/base_link.STL
Joints:
- added joint FL_foot_joint: type fixed, parent FL_calf_link, child FL_foot_link, origin xyz=0 0 -0.21577 rpy=0 0 0, axis 0 0 0
- added joint FR_foot_joint: type fixed, parent FR_calf_link, child FR_foot_link, origin xyz=0 0 -0.21574 rpy=0 0 0, axis 0 0 0
- added joint RL_foot_joint: type fixed, parent RL_calf_link, child RL_foot_link, origin xyz=0 0 -0.21577 rpy=0 0 0, axis 0 0 0
- added joint RR_foot_joint: type fixed, parent RR_calf_link, child RR_foot_link, origin xyz=0 0 -0.21577 rpy=0 0 0, axis 0 0 0
- joint FL_calf_joint: origin xyz=-0.17504 -0.001 -0.11602 rpy=3.1416 -1.3726 -3.1416 -> xyz=-0.19288 0.001 0.083055 rpy=-3.1416 -1.1642 0
- joint FL_hip_joint: origin xyz=0.209 0.0575 0 rpy=-0.20776 0 0 -> xyz=0.209 0.0575 0 rpy=0 0 0
- joint FL_thigh_joint: axis 0 1 0 -> 0 -1 0; origin xyz=0 0.0975 0 rpy=0 -0.77573 0 -> xyz=0 0.0975 0 rpy=-3.1416 -1.1642 0
- joint FR_calf_joint: origin xyz=0 -0.001 -0.21 rpy=3.1416 -0.38712 0 -> xyz=0 -0.001 -0.21 rpy=0 0 -3.1416
- joint FR_hip_joint: origin xyz=0.209 -0.0575 0 rpy=-0.079471 0 0 -> xyz=0.209 -0.0575 0 rpy=0 0 0
- joint FR_thigh_joint: origin xyz=0 -0.0975 0 rpy=0 -1.3591 3.1416 -> xyz=0 -0.10672 0 rpy=0 0 3.1416
- joint RL_calf_joint: origin xyz=0.046814 -0.001 -0.20472 rpy=-3.1416 -0.16231 3.1416 -> xyz=0.0082591 0.001 -0.20984 rpy=0 0.039339 3.1416
- joint RL_hip_joint: origin xyz=-0.212 0.0575 0 rpy=0.20476 0 0 -> xyz=-0.212 0.0575 0 rpy=0 0 0
- joint RL_thigh_joint: origin xyz=0 -0.0975 0 rpy=0 1.463 0 -> xyz=0 -0.0975 0 rpy=0 0 0
- joint RR_calf_joint: origin xyz=0 0.001 -0.21 rpy=3.1416 -0.38712 -3.1416 -> xyz=0 0.001 -0.21 rpy=0 0 0

Commit message: first

File: urdf/ASK-4.urdf (robot description, URDF)
Before this commit: robot ASK-4-2, 17 links, 15 joints
Links:
- link FL_calf_link: mass 0.196508884495562 -> 0.19650888449556; geometry collision mesh filename=package://ASK-4-3/meshes/FL_calf_link.STL; visual mesh filename=package://ASK-4-3/meshes/FL_calf_link.STL
- link FL_foot_link: geometry collision mesh filename=package://ASK-4-3/meshes/FL_foot_link.STL; visual mesh filename=package://ASK-4-3/meshes/FL_foot_link.STL
- link FL_hip_link: geometry collision mesh filename=package://ASK-4-3/meshes/FL_hip_link.STL; visual mesh filename=package://ASK-4-3/meshes/FL_hip_link.STL
- link FL_thigh_link: mass 0.98851736736006 -> 0.988517367360061; geometry collision mesh filename=package://ASK-4-3/meshes/FL_thigh_link.STL; visual mesh filename=package://ASK-4-3/meshes/FL_thigh_link.STL
- link FR_calf_link: mass 0.196508884495563 -> 0.196508884495562; geometry collision mesh filename=package://ASK-4-3/meshes/FR_calf_link.STL; visual mesh filename=package://ASK-4-3/meshes/FR_calf_link.STL
- link FR_foot_link: mass 0.0332506166455944 -> 0.0332506166455943; geometry collision mesh filename=package://ASK-4-3/meshes/FR_foot_link.STL; visual mesh filename=package://ASK-4-3/meshes/FR_foot_link.STL
- link FR_hip_link: geometry collision mesh filename=package://ASK-4-3/meshes/FR_hip_link.STL; visual mesh filename=package://ASK-4-3/meshes/FR_hip_link.STL
- link FR_thigh_link: mass 0.981796539065317 -> 0.981796539065316; geometry collision mesh filename=package://ASK-4-3/meshes/FR_thigh_link.STL; visual mesh filename=package://ASK-4-3/meshes/FR_thigh_link.STL
- link RL_calf_link: geometry collision mesh filename=package://ASK-4-3/meshes/RL_calf_link.STL; visual mesh filename=package://ASK-4-3/meshes/RL_calf_link.STL
- link RL_foot_link: geometry collision mesh filename=package://ASK-4-3/meshes/RL_foot_link.STL; visual mesh filename=package://ASK-4-3/meshes/RL_foot_link.STL
- link RL_hip_link: geometry collision mesh filename=package://ASK-4-3/meshes/RL_hip_link.STL; visual mesh filename=package://ASK-4-3/meshes/RL_hip_link.STL
- link RL_thigh_link: mass 0.988547565628563 -> 0.988547565363266; geometry collision mesh filename=package://ASK-4-3/meshes/RL_thigh_link.STL; visual mesh filename=package://ASK-4-3/meshes/RL_thigh_link.STL
- link RR_calf_link: mass 0.196508883743766 -> 0.196508884495562; geometry collision mesh filename=package://ASK-4-3/meshes/RR_calf_link.STL; visual mesh filename=package://ASK-4-3/meshes/RR_calf_link.STL
- link RR_foot_link: geometry collision mesh filename=package://ASK-4-3/meshes/RR_foot_link.STL; visual mesh filename=package://ASK-4-3/meshes/RR_foot_link.STL
- link RR_hip_link: geometry collision mesh filename=package://ASK-4-3/meshes/RR_hip_link.STL; visual mesh filename=package://ASK-4-3/meshes/RR_hip_link.STL
- link RR_thigh_link: mass 0.981796539186015 -> 0.981796539396402; geometry collision mesh filename=package://ASK-4-3/meshes/RR_thigh_link.STL; visual mesh filename=package://ASK-4-3/meshes/RR_thigh_link.STL
- link base_link: geometry collision mesh filename=package://ASK-4-3/meshes/base_link.STL; visual mesh filename=package://ASK-4-3/meshes/base_link.STL
Joints:
- added joint RR_thigh_joint: type revolute, parent RR_hip_link, child RR_thigh_link, origin xyz=0 -0.0975 0 rpy=0 0 0, axis 0 -1 0, limit lower=-3.14 upper=3.14 effort=100 velocity=100
- joint FL_calf_joint: origin xyz=-0.19288 0.001 0.083055 rpy=-3.1416 -1.1642 0 -> xyz=0 -0.001 -0.21 rpy=0 0 0
- joint FL_thigh_joint: axis 0 -1 0 -> 0 1 0; origin xyz=0 0.0975 0 rpy=-3.1416 -1.1642 0 -> xyz=0 0.0975 0 rpy=0 0 0
- joint FR_calf_joint: origin xyz=0 -0.001 -0.21 rpy=0 0 -3.1416 -> xyz=0 0.001 -0.21 rpy=0 0 0
- joint FR_thigh_joint: axis 0 1 0 -> 0 -1 0; origin xyz=0 -0.10672 0 rpy=0 0 3.1416 -> xyz=0 -0.10672 0 rpy=0 0 0
- joint RL_thigh_joint: child RR_thigh_link -> RL_thigh_link; limit lower=-3.14 upper=3.14 effort=100 velocity=100 -> lower=0 upper=0 effort=0 velocity=0; origin xyz=0 -0.0975 0 rpy=0 0 0 -> xyz=0 0.0975 0 rpy=0 0.039339 3.1416; parent RR_hip_link -> RL_hip_link
- joint RR_hip_joint: origin xyz=-0.212 -0.0575 0 rpy=0 0 0 -> xyz=-0.212000000000005 -0.057499999999997 0 rpy=0 0 0

Commit message: first

File: urdf/ASK-4.urdf (robot description, URDF)
Before this commit: robot ASK-4-3, 17 links, 16 joints
Links:
- link FL_calf_link: geometry collision mesh filename=package://ASK-4-5/meshes/FL_calf_link.STL; visual mesh filename=package://ASK-4-5/meshes/FL_calf_link.STL
- link FL_foot_link: geometry collision mesh filename=package://ASK-4-5/meshes/FL_foot_link.STL; visual mesh filename=package://ASK-4-5/meshes/FL_foot_link.STL
- link FL_hip_link: geometry collision mesh filename=package://ASK-4-5/meshes/FL_hip_link.STL; visual mesh filename=package://ASK-4-5/meshes/FL_hip_link.STL
- link FL_thigh_link: mass 0.988517367360061 -> 0.988517367587917; geometry collision mesh filename=package://ASK-4-5/meshes/FL_thigh_link.STL; visual mesh filename=package://ASK-4-5/meshes/FL_thigh_link.STL
- link FR_calf_link: geometry collision mesh filename=package://ASK-4-5/meshes/FR_calf_link.STL; visual mesh filename=package://ASK-4-5/meshes/FR_calf_link.STL
- link FR_foot_link: mass 0.0332506166455943 -> 0.0332506166455944; geometry collision mesh filename=package://ASK-4-5/meshes/FR_foot_link.STL; visual mesh filename=package://ASK-4-5/meshes/FR_foot_link.STL
- link FR_hip_link: geometry collision mesh filename=package://ASK-4-5/meshes/FR_hip_link.STL; visual mesh filename=package://ASK-4-5/meshes/FR_hip_link.STL
- link FR_thigh_link: mass 0.981796539065316 -> 0.981796539065315; geometry collision mesh filename=package://ASK-4-5/meshes/FR_thigh_link.STL; visual mesh filename=package://ASK-4-5/meshes/FR_thigh_link.STL
- link RL_calf_link: geometry collision mesh filename=package://ASK-4-5/meshes/RL_calf_link.STL; visual mesh filename=package://ASK-4-5/meshes/RL_calf_link.STL
- link RL_foot_link: geometry collision mesh filename=package://ASK-4-5/meshes/RL_foot_link.STL; visual mesh filename=package://ASK-4-5/meshes/RL_foot_link.STL
- link RL_hip_link: geometry collision mesh filename=package://ASK-4-5/meshes/RL_hip_link.STL; visual mesh filename=package://ASK-4-5/meshes/RL_hip_link.STL
- link RL_thigh_link: mass 0.988547565363266 -> 0.988547565628561; geometry collision mesh filename=package://ASK-4-5/meshes/RL_thigh_link.STL; visual mesh filename=package://ASK-4-5/meshes/RL_thigh_link.STL
- link RR_calf_link: mass 0.196508884495562 -> 0.196508884495561; geometry collision mesh filename=package://ASK-4-5/meshes/RR_calf_link.STL; visual mesh filename=package://ASK-4-5/meshes/RR_calf_link.STL
- link RR_foot_link: geometry collision mesh filename=package://ASK-4-5/meshes/RR_foot_link.STL; visual mesh filename=package://ASK-4-5/meshes/RR_foot_link.STL
- link RR_hip_link: geometry collision mesh filename=package://ASK-4-5/meshes/RR_hip_link.STL; visual mesh filename=package://ASK-4-5/meshes/RR_hip_link.STL
- link RR_thigh_link: mass 0.981796539396402 -> 0.981796539396403; geometry collision mesh filename=package://ASK-4-5/meshes/RR_thigh_link.STL; visual mesh filename=package://ASK-4-5/meshes/RR_thigh_link.STL
- link base_link: geometry collision mesh filename=package://ASK-4-5/meshes/base_link.STL; visual mesh filename=package://ASK-4-5/meshes/base_link.STL
Joints:
- joint FL_calf_joint: origin xyz=0 -0.001 -0.21 rpy=0 0 0 -> xyz=0.192877994043746 -0.00100000000000014 0.0830546772533787 rpy=-3.14159265358979 -1.16418582684397 3.14159265358979
- joint FL_foot_joint: origin xyz=0 0 -0.21577 rpy=0 0 0 -> xyz=0 0 -0.215773231361156 rpy=0 0 0
- joint FL_hip_joint: origin xyz=0.209 0.0575 0 rpy=0 0 0 -> xyz=0.209 0.0575000000000031 0 rpy=0 0 0
- joint FL_thigh_joint: origin xyz=0 0.0975 0 rpy=0 0 0 -> xyz=0 0.0975 0 rpy=3.14159265358979 1.16418582684397 3.14159265358979
- joint FR_calf_joint: origin xyz=0 0.001 -0.21 rpy=0 0 0 -> xyz=0 0.00100000000000315 -0.210000000000006 rpy=0 0 0
- joint FR_foot_joint: origin xyz=0 0 -0.21574 rpy=0 0 0 -> xyz=0 0 -0.21574063533816 rpy=0 0 0
- joint FR_hip_joint: origin xyz=0.209 -0.0575 0 rpy=0 0 0 -> xyz=0.209000000000005 -0.0574999999999968 0 rpy=0 0 0
- joint FR_thigh_joint: origin xyz=0 -0.10672 0 rpy=0 0 0 -> xyz=0 -0.0975 0 rpy=0 0 0
- joint RL_calf_joint: origin xyz=0.0082591 0.001 -0.20984 rpy=0 0.039339 3.1416 -> xyz=0.00825912262911521 0.00100000000000011 -0.209837524988716 rpy=0 0.0393393013816893 3.14159265358979
- joint RL_foot_joint: origin xyz=0 0 -0.21577 rpy=0 0 0 -> xyz=0 0 -0.215773231361156 rpy=0 0 0
- joint RL_hip_joint: origin xyz=-0.212 0.0575 0 rpy=0 0 0 -> xyz=-0.212 0.0575000000000033 0 rpy=0 0 0
- joint RL_thigh_joint: origin xyz=0 0.0975 0 rpy=0 0.039339 3.1416 -> xyz=0 0.0974999999999997 0 rpy=0 0.0393393013816893 3.14159265358979
- joint RR_calf_joint: origin xyz=0 0.001 -0.21 rpy=0 0 0 -> xyz=0 0.00100000000000035 -0.210000000000027 rpy=0 0 0
- joint RR_foot_joint: origin xyz=0 0 -0.21577 rpy=0 0 0 -> xyz=0 0 -0.215773231361156 rpy=0 0 0

Commit message: first

File: urdf/ASK-4.urdf (robot description, URDF)
Before this commit: robot ASK-4-5, 17 links, 16 joints
Links:
- link FL_calf_link: geometry collision mesh filename=package://ASK-4-3/meshes/FL_calf_link.STL; visual mesh filename=package://ASK-4-3/meshes/FL_calf_link.STL
- link FL_foot_link: geometry collision mesh filename=package://ASK-4-3/meshes/FL_foot_link.STL; visual mesh filename=package://ASK-4-3/meshes/FL_foot_link.STL
- link FL_hip_link: geometry collision mesh filename=package://ASK-4-3/meshes/FL_hip_link.STL; visual mesh filename=package://ASK-4-3/meshes/FL_hip_link.STL
- link FL_thigh_link: mass 0.988517367587917 -> 0.988517367360061; geometry collision mesh filename=package://ASK-4-3/meshes/FL_thigh_link.STL; visual mesh filename=package://ASK-4-3/meshes/FL_thigh_link.STL
- link FR_calf_link: geometry collision mesh filename=package://ASK-4-3/meshes/FR_calf_link.STL; visual mesh filename=package://ASK-4-3/meshes/FR_calf_link.STL
- link FR_foot_link: mass 0.0332506166455944 -> 0.0332506166455943; geometry collision mesh filename=package://ASK-4-3/meshes/FR_foot_link.STL; visual mesh filename=package://ASK-4-3/meshes/FR_foot_link.STL
- link FR_hip_link: geometry collision mesh filename=package://ASK-4-3/meshes/FR_hip_link.STL; visual mesh filename=package://ASK-4-3/meshes/FR_hip_link.STL
- link FR_thigh_link: mass 0.981796539065315 -> 0.981796539065316; geometry collision mesh filename=package://ASK-4-3/meshes/FR_thigh_link.STL; visual mesh filename=package://ASK-4-3/meshes/FR_thigh_link.STL
- link RL_calf_link: geometry collision mesh filename=package://ASK-4-10/meshes/RL_calf_link.STL; visual mesh filename=package://ASK-4-10/meshes/RL_calf_link.STL
- link RL_foot_link: geometry collision mesh filename=package://ASK-4-10/meshes/RL_foot_link.STL; visual mesh filename=package://ASK-4-10/meshes/RL_foot_link.STL
- link RL_hip_link: geometry collision mesh filename=package://ASK-4-10/meshes/RL_hip_link.STL; visual mesh filename=package://ASK-4-10/meshes/RL_hip_link.STL
- link RL_thigh_link: mass 0.988547565628561 -> 0.988547565363266; geometry collision mesh filename=package://ASK-4-10/meshes/RL_thigh_link.STL; visual mesh filename=package://ASK-4-10/meshes/RL_thigh_link.STL
- link RR_calf_link: mass 0.196508884495561 -> 0.196508884495562; geometry collision mesh filename=package://ASK-4-3/meshes/RR_calf_link.STL; visual mesh filename=package://ASK-4-3/meshes/RR_calf_link.STL
- link RR_foot_link: geometry collision mesh filename=package://ASK-4-3/meshes/RR_foot_link.STL; visual mesh filename=package://ASK-4-3/meshes/RR_foot_link.STL
- link RR_hip_link: geometry collision mesh filename=package://ASK-4-3/meshes/RR_hip_link.STL; visual mesh filename=package://ASK-4-3/meshes/RR_hip_link.STL
- link RR_thigh_link: mass 0.981796539396403 -> 0.981796539396402; geometry collision mesh filename=package://ASK-4-3/meshes/RR_thigh_link.STL; visual mesh filename=package://ASK-4-3/meshes/RR_thigh_link.STL
- link base_link: geometry collision mesh filename=package://ASK-4-3/meshes/base_link.STL; visual mesh filename=package://ASK-4-3/meshes/base_link.STL
Joints:
- joint FL_calf_joint: origin xyz=0.192877994043746 -0.00100000000000014 0.0830546772533787 rpy=-3.14159265358979 -1.16418582684397 3.14159265358979 -> xyz=0 -0.001 -0.21 rpy=0 0 0
- joint FL_foot_joint: origin xyz=0 0 -0.215773231361156 rpy=0 0 0 -> xyz=0 0 -0.21577 rpy=0 0 0
- joint FL_hip_joint: origin xyz=0.209 0.0575000000000031 0 rpy=0 0 0 -> xyz=0.209 0.0575 0 rpy=0 0 0
- joint FL_thigh_joint: origin xyz=0 0.0975 0 rpy=3.14159265358979 1.16418582684397 3.14159265358979 -> xyz=0 0.0975 0 rpy=0 0 0
- joint FR_calf_joint: origin xyz=0 0.00100000000000315 -0.210000000000006 rpy=0 0 0 -> xyz=0 0.001 -0.21 rpy=0 0 0
- joint FR_foot_joint: origin xyz=0 0 -0.21574063533816 rpy=0 0 0 -> xyz=0 0 -0.21574 rpy=0 0 0
- joint FR_hip_joint: origin xyz=0.209000000000005 -0.0574999999999968 0 rpy=0 0 0 -> xyz=0.209 -0.0575 0 rpy=0 0 0
- joint FR_thigh_joint: origin xyz=0 -0.0975 0 rpy=0 0 0 -> xyz=0 -0.10672 0 rpy=0 0 0
- joint RL_calf_joint: axis 0 -1 0 -> 0 1 0; origin xyz=0.00825912262911521 0.00100000000000011 -0.209837524988716 rpy=0 0.0393393013816893 3.14159265358979 -> xyz=-0.00825912262911466 -0.00100000000000011 -0.209837524988717 rpy=0 0.0393393013816893 0
- joint RL_thigh_joint: axis 0 -1 0 -> 0 1 0; origin xyz=0 0.0974999999999997 0 rpy=0 0.0393393013816893 3.14159265358979 -> xyz=0 0.0974999999999997 0 rpy=0 -0.0393393013816893 0
- joint RR_calf_joint: origin xyz=0 0.00100000000000035 -0.210000000000027 rpy=0 0 0 -> xyz=0 0.001 -0.21 rpy=0 0 0
- joint RR_foot_joint: origin xyz=0 0 -0.215773231361156 rpy=0 0 0 -> xyz=0 0 -0.21577 rpy=0 0 0

Commit message: first

File: urdf/ASK-4.urdf (robot description, URDF)
Before this commit: robot ASK-4-3, 17 links, 16 joints
Links:
- link FL_calf_link: geometry collision mesh filename=package://urdf_tutorial/meshes/FL_calf_link.STL; visual mesh filename=package://urdf_tutorial/meshes/FL_calf_link.STL
- link FL_hip_link: geometry collision mesh filename=package://urdf_tutorial/meshes/FL_hip_link.STL; visual mesh filename=package://urdf_tutorial/meshes/FL_hip_link.STL
- link FL_thigh_link: geometry collision mesh filename=package://urdf_tutorial/meshes/FL_thigh_link.STL; visual mesh filename=package://urdf_tutorial/meshes/FL_thigh_link.STL
- link base_link: geometry collision mesh filename=package://urdf_tutorial/meshes/base_link.STL; visual mesh filename=package://urdf_tutorial/meshes/base_link.STL

Commit message: first

File: urdf/ASK-4.urdf (robot description, URDF)
Before this commit: robot ASK-4-3, 18 links, 17 joints
Links:
- link FL_calf_link: mass 0.19650888449556 -> 0.1965110
- link FL_foot_link: mass 0.0332506166455944 -> 0.0338791
- link FL_hip_link: mass 0.337654873921649 -> 0.3376556
- link FL_thigh_link: mass 0.988517367360061 -> 0.9885170
- link FR_calf_link: mass 0.196508884495562 -> 0.1965110
- link FR_foot_link: mass 0.0332506166455943 -> 0.0338791
- link FR_hip_link: mass 0.337657104489193 -> 0.3376577
- link FR_thigh_link: mass 0.981796539065316 -> 0.9885170
- link RL_calf_link: mass 0.196508884495564 -> 0.1965110
- link RL_foot_link: mass 0.0332506166455944 -> 0.0338791
- link RL_hip_link: mass 0.33765486830875 -> 0.3376556
- link RL_thigh_link: mass 0.988547565363266 -> 0.9885170
- link RR_calf_link: mass 0.196508884495562 -> 0.1965110
- link RR_foot_link: mass 0.0332506166455944 -> 0.0338791
- link RR_hip_link: mass 0.337657104489195 -> 0.3376556
- link RR_thigh_link: mass 0.981796539396402 -> 0.9885170
- link base_link: mass 5.13967166144139 -> 4.3155061
