Commit message: first

File: urdf/ASK-4.urdf (robot description, URDF)
Before this commit: robot ASK-4-3, 17 links, 16 joints
Links:
- added link dummy_link
- link FL_calf_link: geometry collision mesh filename=package://urdf_tutorial/meshes/calf_link.STL; visual mesh filename=package://urdf_tutorial/meshes/calf_link.STL
- link FL_foot_link: geometry collision mesh filename=package://urdf_tutorial/meshes/foot_link.STL; visual mesh filename=package://urdf_tutorial/meshes/foot_link.STL
- link FL_hip_link: geometry collision mesh filename=package://urdf_tutorial/meshes/hip_link.STL; visual mesh filename=package://urdf_tutorial/meshes/hip_link.STL
- link FL_thigh_link: geometry collision mesh filename=package://urdf_tutorial/meshes/thigh_link.STL; visual mesh filename=package://urdf_tutorial/meshes/thigh_link.STL
- link FR_calf_link: geometry collision mesh filename=package://urdf_tutorial/meshes/calf_link.STL; visual mesh filename=package://urdf_tutorial/meshes/calf_link.STL
- link FR_foot_link: geometry collision mesh filename=package://urdf_tutorial/meshes/foot_link.STL; visual mesh filename=package://urdf_tutorial/meshes/foot_link.STL
- link FR_hip_link: geometry collision mesh filename=package://urdf_tutorial/meshes/R_hip_link.STL; visual mesh filename=package://urdf_tutorial/meshes/R_hip_link.STL
- link FR_thigh_link: geometry collision mesh filename=package://urdf_tutorial/meshes/R_thigh_link.STL; visual mesh filename=package://urdf_tutorial/meshes/R_thigh_link.STL
- link RL_calf_link: geometry collision mesh filename=package://urdf_tutorial/meshes/calf_link.STL; visual mesh filename=package://urdf_tutorial/meshes/calf_link.STL
- link RL_foot_link: geometry collision mesh filename=package://urdf_tutorial/meshes/foot_link.STL; visual mesh filename=package://urdf_tutorial/meshes/foot_link.STL
- link RL_hip_link: geometry collision mesh filename=package://urdf_tutorial/meshes/hip_link.STL; visual mesh filename=package://urdf_tutorial/meshes/hip_link.STL
- link RL_thigh_link: geometry collision mesh filename=package://urdf_tutorial/meshes/thigh_link.STL; visual mesh filename=package://urdf_tutorial/meshes/thigh_link.STL
- link RR_calf_link: geometry collision mesh filename=package://urdf_tutorial/meshes/calf_link.STL; visual mesh filename=package://urdf_tutorial/meshes/calf_link.STL
- link RR_foot_link: geometry collision mesh filename=package://urdf_tutorial/meshes/foot_link.STL; visual mesh filename=package://urdf_tutorial/meshes/foot_link.STL
- link RR_hip_link: geometry collision mesh filename=package://urdf_tutorial/meshes/R_hip_link.STL; visual mesh filename=package://urdf_tutorial/meshes/R_hip_link.STL
- link RR_thigh_link: geometry collision mesh filename=package://urdf_tutorial/meshes/R_thigh_link.STL; visual mesh filename=package://urdf_tutorial/meshes/R_thigh_link.STL
Joints:
- added joint dummy_joint: type fixed, parent dummy_link, child base_link

Commit message: first

File: urdf/ASK-4.urdf (robot description, URDF)
Before this commit: robot ASK-4-3, 18 links, 17 joints
Links:
- link FL_calf_link: geometry collision box size=0.21 0.013 0.0252; visual mesh filename=package://urdf_tutorial/meshes/calf_link.STL
- link FL_foot_link: geometry collision sphere radius=0.021; visual mesh filename=package://urdf_tutorial/meshes/foot_link.STL
- link FL_hip_link: geometry collision cylinder length=0.082 radius=0.05; visual mesh filename=package://urdf_tutorial/meshes/hip_link.STL
- link FL_thigh_link: geometry collision box size=0.18 0.0278 0.034; visual mesh filename=package://urdf_tutorial/meshes/thigh_link.STL
- link FR_calf_link: geometry collision box size=0.21 0.013 0.0252; visual mesh filename=package://urdf_tutorial/meshes/calf_link.STL
- link FR_foot_link: geometry collision sphere radius=0.021; visual mesh filename=package://urdf_tutorial/meshes/foot_link.STL
- link FR_hip_link: geometry collision cylinder length=0.082 radius=0.05; visual mesh filename=package://urdf_tutorial/meshes/R_hip_link.STL
- link FR_thigh_link: geometry collision box size=0.18 0.0278 0.034; visual mesh filename=package://urdf_tutorial/meshes/R_thigh_link.STL
- link RL_calf_link: geometry collision box size=0.21 0.013 0.0252; visual mesh filename=package://urdf_tutorial/meshes/calf_link.STL
- link RL_foot_link: geometry collision sphere radius=0.021; visual mesh filename=package://urdf_tutorial/meshes/foot_link.STL
- link RL_hip_link: geometry collision cylinder length=0.082 radius=0.05; visual mesh filename=package://urdf_tutorial/meshes/hip_link.STL
- link RL_thigh_link: geometry collision box size=0.18 0.0278 0.034; visual mesh filename=package://urdf_tutorial/meshes/thigh_link.STL
- link RR_calf_link: geometry collision box size=0.21 0.013 0.0252; visual mesh filename=package://urdf_tutorial/meshes/calf_link.STL
- link RR_foot_link: geometry collision sphere radius=0.021; visual mesh filename=package://urdf_tutorial/meshes/foot_link.STL
- link RR_hip_link: geometry collision cylinder length=0.082 radius=0.05; visual mesh filename=package://urdf_tutorial/meshes/R_hip_link.STL
- link RR_thigh_link: geometry collision box size=0.18 0.0278 0.034; visual mesh filename=package://urdf_tutorial/meshes/R_thigh_link.STL
- link base_link: geometry collision box size=0.306 0.22 0.14; visual mesh filename=package://urdf_tutorial/meshes/base_link.STL
Joints:
- joint FL_calf_joint: origin xyz=0 -0.001 -0.21 rpy=0 0 0 -> xyz=0 0 -0.21 rpy=0 0 0
- joint FR_calf_joint: origin xyz=0 0.001 -0.21 rpy=0 0 0 -> xyz=0 0.00 -0.21 rpy=0 0 0
- joint RL_calf_joint: limit lower=0 upper=0 effort=0 velocity=0 -> lower=-3.14 upper=3.14 effort=100 velocity=100; origin xyz=-0.00825912262911466 -0.00100000000000011 -0.209837524988717 rpy=0 0.0393393013816893 0 -> xyz=0 0 -0.209837524988717 rpy=0 0 0
- joint RL_hip_joint: origin xyz=-0.212 0.0575000000000033 0 rpy=0 0 0 -> xyz=-0.212 0.0575 0 rpy=0 0 0
- joint RL_thigh_joint: limit lower=0 upper=0 effort=0 velocity=0 -> lower=3.14 upper=-3.14 effort=100 velocity=100; origin xyz=0 0.0974999999999997 0 rpy=0 -0.0393393013816893 0 -> xyz=0 0.0974999999999997 0 rpy=0 0 0
- joint RR_calf_joint: origin xyz=0 0.001 -0.21 rpy=0 0 0 -> xyz=0 0.00 -0.21 rpy=0 0 0
- joint RR_hip_joint: origin xyz=-0.212000000000005 -0.057499999999997 0 rpy=0 0 0 -> xyz=-0.212000000000005 -0.0575 0 rpy=0 0 0

Commit message: first

File: urdf/ASK-4.urdf (robot description, URDF)
Before this commit: robot ASK-4-3, 18 links, 17 joints
Links:
- added link bottom; collision box size=0.04 0.16 0.12
- added link head; collision box size=0.04 0.16 0.12
- link FR_thigh_link: mass 0.9885170 -> 0.98817966
- link RL_thigh_link: mass 0.9885170 -> 0.9885474
- link RR_hip_link: mass 0.3376556 -> 0.3376577
- link RR_thigh_link: mass 0.9885170 -> 0.9817966
Joints:
- added joint bottom_joint: type fixed, parent base_link, child bottom, origin xyz=-0.34734 0 0 rpy=0 0 0
- added joint head_joint: type fixed, parent base_link, child head, origin xyz=0.34734 0 0 rpy=0 0 0

Commit message: first

File: urdf/ASK-4.urdf (robot description, URDF)
Before this commit: robot ASK-4-3, 20 links, 19 joints
Joints:
- joint FL_calf_joint: axis 0 -1 0 -> 0 1 0
- joint FR_calf_joint: axis 0 -1 0 -> 0 1 0
- joint FR_thigh_joint: axis 0 -1 0 -> 0 1 0
- joint RL_thigh_joint: limit lower=3.14 upper=-3.14 effort=100 velocity=100 -> lower=-3.14 upper=3.14 effort=100 velocity=100; origin xyz=0 0.0974999999999997 0 rpy=0 0 0 -> xyz=0 0.0975 0 rpy=0 0 0
- joint RR_calf_joint: axis 0 -1 0 -> 0 1 0
- joint RR_thigh_joint: axis 0 -1 0 -> 0 1 0
