Commit message: first

File: urdf/2.urdf (robot description, URDF)
Before this commit: robot ASK-4-3, 21 links, 20 joints
Links:
- link FL_calf_link: geometry collision box size=0.21 0.013 0.0252; visual mesh filename=../meshes/calf_link.STL
- link FL_foot: geometry collision sphere radius=0.021; visual mesh filename=../meshes/foot_link.STL
- link FL_hip_link: geometry collision cylinder length=0.082 radius=0.05; visual mesh filename=../meshes/hip_link.STL
- link FL_thigh_link: geometry collision box size=0.18 0.0278 0.034; visual mesh filename=../meshes/thigh_link.STL
- link FR_calf_link: geometry collision box size=0.21 0.013 0.0252; visual mesh filename=../meshes/calf_link.STL
- link FR_foot: geometry collision sphere radius=0.021; visual mesh filename=../meshes/foot_link.STL
- link FR_hip_link: geometry collision cylinder length=0.082 radius=0.05; visual mesh filename=../meshes/R_hip_link.STL
- link FR_thigh_link: geometry collision box size=0.18 0.0278 0.034; visual mesh filename=../meshes/R_thigh_link.STL
- link RL_calf_link: geometry collision box size=0.21 0.013 0.0252; visual mesh filename=../meshes/calf_link.STL
- link RL_foot: geometry collision sphere radius=0.021; visual mesh filename=../meshes/foot_link.STL
- link RL_hip_link: geometry collision cylinder length=0.082 radius=0.05; visual mesh filename=../meshes/hip_link.STL
- link RL_thigh_link: geometry collision box size=0.18 0.0278 0.034; visual mesh filename=../meshes/thigh_link.STL
- link RR_calf_link: geometry collision box size=0.21 0.013 0.0252; visual mesh filename=../meshes/calf_link.STL
- link RR_foot: geometry collision sphere radius=0.021; visual mesh filename=../meshes/foot_link.STL
- link RR_hip_link: geometry collision cylinder length=0.082 radius=0.05; visual mesh filename=../meshes/R_hip_link.STL
- link RR_thigh_link: geometry collision box size=0.18 0.0278 0.034; visual mesh filename=../meshes/R_thigh_link.STL
- link base_link: geometry collision box size=0.306 0.22 0.14; visual mesh filename=../meshes/base_link.STL
Joints:
- joint FL_calf_joint: axis 0 1 0 -> 0 -1 0
- joint FR_calf_joint: axis 0 1 0 -> 0 -1 0
- joint FR_thigh_joint: axis 0 1 0 -> 0 -1 0
- joint RL_thigh_joint: limit lower=-3.14 upper=3.14 effort=100 velocity=100 -> lower=3.14 upper=-3.14 effort=100 velocity=100; origin xyz=0 0.0975 0 rpy=0 0 0 -> xyz=0 0.0974999999999997 0 rpy=0 0 0
- joint RR_calf_joint: axis 0 1 0 -> 0 -1 0
- joint RR_thigh_joint: axis 0 1 0 -> 0 -1 0
